File: examples/06-intelligent-placement/fixtures/mcu_board.kicad_pcb (KiCad board)
At the start: 2 copper layers, 80 x 70 mm, 17 parts, among them J1 USB-C, SW1 RESET, U1 STM32F103, U2 AMS1117-3.3, Y1 8MHz

Commit message: chore: Remove obsolete ISSUES-FOUND.md
All issues from v0.7.1 testing have been verified as fixed:
- #438 analyze signal-integrity: now implemented
- #439 parts availability: no more IndexError
- #440 router --grid: parameter now respected
- #441 net-status: via-to-zone detection working
- #442 audit: no more attribute errors
- #443 estimate cost: shows component costs
- #444 reasoning: correct board size, layers, pad names
- #445 placement --format json: now supported
- #446 router --layers: multi-layer support working
- #447 validate --sync: accepts positional arguments

🤖 Generated with [Claude Code](https://claude.com/claude-code)

Co-Authored-By: Claude Opus 4.5 <noreply@anthropic.com>
Parts:
- moved C3 20.3 mm to (127.2, 138.3)
- moved U2 17.8 mm to (118.7, 122.6)
- moved C6 15.6 mm to (137.3, 142.8)
- moved TP2 12.0 mm to (163.4, 138.1)
- moved C5 9.98 mm to (117.5, 136.8)
- moved SW1 9.53 mm to (162.7, 118.9)
- moved C4 9.25 mm to (140.4, 112.5)
- moved TP1 8.80 mm to (155.4, 142.5)
- moved C2 7.73 mm to (157.4, 132.4)
- moved C1 6.05 mm to (150.6, 114.0)
- moved U1 4.84 mm to (142.6, 129.1)
- moved Y1 2.43 mm to (127.9, 113.8)
