File: boards/external/chorus-test-revA/chorus-test-revA_routed.kicad_pcb (KiCad board)
At the start: 4 copper layers, 65 x 56 mm, 38 parts, among them J2 RPi_GPIO, J3 Audio_Out, J4 SWD, U3 74LVC1G17, U4 XC6206-3.3V, U5 XC6206-3.3V, U6 PCM5122PW, U7 74LVC1G17, U8 STM32C011F4P6, Y2 24.576MHz

Commit message: fix(chorus): correct PCM5122 PCB pad net assignments to match TSSOP-28 datasheet
The PCB had I2S signals (BCLK, LRCLK, DIN) assigned to charge pump
pads 3-5 instead of their correct I2S interface pads 21-23. This
would route digital audio signals to the charge pump circuit, which
would damage the IC or prevent operation. Also corrects power (DVDD,
AVDD), ground (DGND, AGND, CPGND), I2C (SCL, SDA), MODE, and
address pin assignments across all 28 pads.

Co-Authored-By: Claude Opus 4.6 <noreply@anthropic.com>
Connections:
- U6 pad 10: (no net) -> Net-U6-VCOM
- U6 pad 11: (no net) -> SDA
- U6 pad 12: (no net) -> SCL
- U6 pad 14: GND -> Net-U6-GPIO4
- U6 pad 15: +3.3VA -> Net-U6-GPIO3
- U6 pad 16: (no net) -> GND
- U6 pad 17: (no net) -> GND
- U6 pad 18: (no net) -> +3.3V
- U6 pad 2: GND -> Net-C19-Pad1
- U6 pad 20: (no net) -> MCLK_DAC
- U6 pad 21: (no net) -> I2S_BCLK
- U6 pad 22: (no net) -> I2S_DIN
- U6 pad 23: (no net) -> I2S_LRCLK
- U6 pad 24: (no net) -> GND
- U6 pad 26: (no net) -> Net-U6-LDOO
- U6 pad 27: (no net) -> GND
- U6 pad 28: GND -> +3.3V
- U6 pad 3: I2S_BCLK -> GNDA
- U6 pad 4: I2S_LRCLK -> Net-C19-Pad2
- U6 pad 5: I2S_DIN -> Net-U6-VNEG
- U6 pad 6: (no net) -> Net-U6-OUTL
- U6 pad 7: (no net) -> Net-U6-OUTR
- U6 pad 8: (no net) -> +3.3VA
- U6 pad 9: (no net) -> GNDA
Changed lines of the file:
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@@
   (net 22 "SYNC_L")
   (net 23 "SYNC_R")
+  (net 24 "SCL")
+  (net 25 "SDA")
+  (net 26 "Net-C19-Pad1")
+  (net 27 "Net-C19-Pad2")
+  (net 28 "Net-U6-VNEG")
+  (net 29 "Net-U6-VCOM")
+  (net 30 "Net-U6-LDOO")
+  (net 31 "Net-U6-GPIO3")
+  (net 32 "Net-U6-GPIO4")
+  (net 33 "Net-U6-OUTL")
+  (net 34 "Net-U6-OUTR")
   (gr_rect
     (start 115.0 75.0)
@@
       (roundrect_rratio 0.25)
       (layers "F.Cu" "F.Paste" "F.Mask")
-      (net 1 "GND")
+      (net 26 "Net-C19-Pad1")
     )
     (pad "3" smd roundrect
@@
       (roundrect_rratio 0.25)
       (layers "F.Cu" "F.Paste" "F.Mask")
-      (net 9 "I2S_BCLK")
+      (net 5 "GNDA")
     )
     (pad "4" smd roundrect
@@
       (roundrect_rratio 0.25)
       (layers "F.Cu" "F.Paste" "F.Mask")
-      (net 10 "I2S_LRCLK")
+      (net 27 "Net-C19-Pad2")
     )
     (pad "5" smd roundrect
@@
       (roundrect_rratio 0.25)
       (layers "F.Cu" "F.Paste" "F.Mask")
-      (net 11 "I2S_DIN")
+      (net 28 "Net-U6-VNEG")
     )
     (pad "6" smd roundrect
@@
       (roundrect_rratio 0.25)
       (layers "F.Cu" "F.Paste" "F.Mask")
+      (net 33 "Net-U6-OUTL")
     )
     (pad "7" smd roundrect
@@
       (roundrect_rratio 0.25)
       (layers "F.Cu" "F.Paste" "F.Mask")
+      (net 34 "Net-U6-OUTR")
     )
     (pad "8" smd roundrect
@@
       (roundrect_rratio 0.25)
       (layers "F.Cu" "F.Paste" "F.Mask")
+      (net 4 "+3.3VA")
     )
     (pad "9" smd roundrect
@@
       (roundrect_rratio 0.25)
       (layers "F.Cu" "F.Paste" "F.Mask")
+      (net 5 "GNDA")
     )
     (pad "10" smd roundrect
@@
       (roundrect_rratio 0.25)
       (layers "F.Cu" "F.Paste" "F.Mask")
+      (net 29 "Net-U6-VCOM")
     )
     (pad "11" smd roundrect
@@
       (roundrect_rratio 0.25)
       (layers "F.Cu" "F.Paste" "F.Mask")
+      (net 25 "SDA")
     )
     (pad "12" smd roundrect
@@
       (roundrect_rratio 0.25)
       (layers "F.Cu" "F.Paste" "F.Mask")
+      (net 24 "SCL")
     )
     (pad "13" smd roundrect
@@
       (roundrect_rratio 0.25)
       (layers "F.Cu" "F.Paste" "F.Mask")
-      (net 1 "GND")
+      (net 32 "Net-U6-GPIO4")
     )
     (pad "15" smd roundrect
@@
       (roundrect_rratio 0.25)
       (layers "F.Cu" "F.Paste" "F.Mask")
-      (net 4 "+3.3VA")
+      (net 31 "Net-U6-GPIO3")
     )
     (pad "16" smd roundrect
@@
       (roundrect_rratio 0.25)
       (layers "F.Cu" "F.Paste" "F.Mask")
+      (net 1 "GND")
     )
     (pad "17" smd roundrect
@@
       (roundrect_rratio 0.25)
       (layers "F.Cu" "F.Paste" "F.Mask")
+      (net 1 "GND")
     )
     (pad "18" smd roundrect
@@
       (roundrect_rratio 0.25)
       (layers "F.Cu" "F.Paste" "F.Mask")
+      (net 3 "+3.3V")
     )
     (pad "19" smd roundrect
@@
       (roundrect_rratio 0.25)
       (layers "F.Cu" "F.Paste" "F.Mask")
+      (net 7 "MCLK_DAC")
     )
     (pad "21" smd roundrect
@@
       (roundrect_rratio 0.25)
       (layers "F.Cu" "F.Paste" "F.Mask")
+      (net 9 "I2S_BCLK")
     )
     (pad "22" smd roundrect
@@
       (roundrect_rratio 0.25)
       (layers "F.Cu" "F.Paste" "F.Mask")
+      (net 11 "I2S_DIN")
     )
     (pad "23" smd roundrect
@@
       (roundrect_rratio 0.25)
       (layers "F.Cu" "F.Paste" "F.Mask")
+      (net 10 "I2S_LRCLK")
     )
     (pad "24" smd roundrect
@@
       (roundrect_rratio 0.25)
       (layers "F.Cu" "F.Paste" "F.Mask")
+      (net 1 "GND")
     )
     (pad "25" smd roundrect
@@
       (roundrect_rratio 0.25)
       (layers "F.Cu" "F.Paste" "F.Mask")
+      (net 30 "Net-U6-LDOO")
     )
     (pad "27" smd roundrect
@@
       (roundrect_rratio 0.25)
       (layers "F.Cu" "F.Paste" "F.Mask")
+      (net 1 "GND")
     )
     (pad "28" smd roundrect
@@
       (roundrect_rratio 0.25)
       (layers "F.Cu" "F.Paste" "F.Mask")
-      (net 1 "GND")
+      (net 3 "+3.3V")
     )
   )
