File: boards/03-usb-joystick/output/usb_joystick_routed.kicad_pcb (KiCad board)
At the start: 2 copper layers, 80 x 60 mm, 12 parts, among them J1 USB-C, J2 Joystick, SW1 Button, SW2 Button, SW3 Button, SW4 Button, U1 MCU, Y1 16MHz

Commit message: fix(board-03): emit missing schematic-side parts in PCB generator + regression test
Issue #2744 (slim scope per curator). The board-03 PCB generator was
silently dropping seven components that the matching schematic emits:

* Y1's 22 pF load caps (C5/C6) -- from
  create_crystal_with_loads(cap_ref_start=5)
* J2's anti-alias filter + BTN pull-up (R10/C10, R11/C11, R12) -- from
  create_analog_joystick(filter_ref_start=10)

Drift caused kct validate --sync to flag seven schematic-only refs and
the BOM<->PCB export preflight to block manufacturing output, even though
the build chain reported "OK verify".

Changes:

* boards/03-usb-joystick/generate_pcb.py:
  - Add generate_resistor() helper for 0402 resistor footprints.
  - Add value= parameter to generate_capacitor() so load caps and filter
    caps can carry the right BOM value ("22pF", "16nF").
  - Add generate_xtal_load_caps() (C5/C6 -> XTAL1/GND, XTAL2/GND).
  - Add generate_joystick_filter() (R10/C10/R11/C11/R12 forming the
    JOY_X/JOY_Y RC filter + JOY_BTN pull-up to VCC).
  - Wire the two helpers into generate_pcb() so every schematic-side
    ref now has a PCB-side footprint.
* boards/03-usb-joystick/route_demo.py: document why USB_CC1/USB_CC2
  skip remains correct -- this demo script uses router.route_all()
  directly and has no layer-escalation path.
* tests/test_board_03_regression.py (new): three regression tests
  pinning (1) all seven refs are present in the regenerated PCB,
  (2) kct validate --sync reports zero errors against the freshly
  regenerated schematic, (3) route_demo.py routes >= 9 signal nets
  fully (matches the curator-specified floor).

Closes #2744
Parts:
- added C10: 16nF, Capacitor_SMD:C_0402_1005Metric, F.Cu at (129.0, 132.5)
- added C11: 16nF, Capacitor_SMD:C_0402_1005Metric, F.Cu at (129.0, 135.0)
- added C5: 22pF, Capacitor_SMD:C_0402_1005Metric, F.Cu at (152.6, 132.0)
- added C6: 22pF, Capacitor_SMD:C_0402_1005Metric, F.Cu at (157.4, 132.0)
- added R10: 10k, Resistor_SMD:R_0402_1005Metric, F.Cu at (127.0, 132.5)
- added R11: 10k, Resistor_SMD:R_0402_1005Metric, F.Cu at (127.0, 135.0)
- added R12: 10k, Resistor_SMD:R_0402_1005Metric, F.Cu at (127.0, 140.0)
Routing:
- net XTAL1: track 18.6 -> 23.7 mm
- net XTAL2: track 0.00 -> 4.11 mm
- net JOY_X: track 23.4 -> 26.8 mm, vias 2 -> 0
- net JOY_BTN: track 28.5 -> 27.3 mm
- net JOY_Y: track 24.7 -> 24.9 mm, vias 2 -> 4
- net BTN2: vias 0 -> 2
