File: boards/01-voltage-divider/output/voltage_divider_routed.kicad_pcb (KiCad board)
At the start: 2 copper layers, 30 x 25 mm, 4 parts, among them J1 Conn_01x02, J2 Conn_01x02

Commit message: fix(router): extend narrow-channel halo to exterior side of same-component plane-net pads (closes #2902)
The 44 `clearance_pad_segment` errors on board-04's U2 west edge originate
in the main router extending escape stubs across F.Cu, clipping plane-net
pads on the same component. No escape-phase predicate could prevent this
(see closed PR #2897 for the diagnostic).

Extends `_apply_narrow_channel_halo` in grid.py to cover the exterior
corridor adjacent to same-component plane-net pads (`pad.net != 0`), in
addition to the existing inter-pad channel coverage from #2879. Width
follows the existing clearance + segment-trace-width margin.

Per-board regression suite re-run; routed PCBs regenerated for boards 01-04.

Closes #2902

Co-Authored-By: Claude Opus 4.7 (1M context) <noreply@anthropic.com>
Routing:
- net GND: track 0.00 -> 24.6 mm, vias 0 -> 1
- net VOUT: track 20.2 -> 10.9 mm, vias 0 -> 1
Other:
- copper layers 2 -> 4
Changed lines of the file:
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@@
   (layers
     (0 "F.Cu" signal)
+    (1 "In1.Cu" signal)
+    (2 "In2.Cu" signal)
     (31 "B.Cu" signal)
     (32 "B.Adhes" user "B.Adhesive")
-    (33 "F.Adhes" user "F.Adhesive")
-    (34 "B.Paste" user)
-    (35 "F.Paste" user)
-    (36 "B.SilkS" user "B.Silkscreen")
-    (37 "F.SilkS" user "F.Silkscreen")
-    (38 "B.Mask" user)
-    (39 "F.Mask" user)
-    (44 "Edge.Cuts" user)
-    (46 "B.CrtYd" user "B.Courtyard")
-    (47 "F.CrtYd" user "F.Courtyard")
-    (48 "B.Fab" user)
-    (49 "F.Fab" user)
+(33 "F.Adhes" user "F.Adhesive")
+(34 "B.Paste" user)
+(35 "F.Paste" user)
+(36 "B.SilkS" user "B.Silkscreen")
+(37 "F.SilkS" user "F.Silkscreen")
+(38 "B.Mask" user)
+(39 "F.Mask" user)
+(44 "Edge.Cuts" user)
+(46 "B.CrtYd" user "B.Courtyard")
+(47 "F.CrtYd" user "F.Courtyard")
+(48 "B.Fab" user)
+(49 "F.Fab" user)
   )
   (setup
@@
   (segment
 		(start 105.0000 111.2300)
-		(end 105.8000 110.4000)
-		(width 0.3)
+		(end 106.5898 111.1898)
+		(width 0.5)
 		(layer "F.Cu")
 		(net 1)
 	)
 	(segment
-		(start 105.8000 110.4000)
-		(end 108.2000 108.0000)
-		(width 0.3)
+		(start 106.5898 111.1898)
+		(end 108.9898 108.7898)
+		(width 0.5)
 		(layer "F.Cu")
 		(net 1)
 	)
 	(segment
-		(start 108.2000 108.0000)
+		(start 108.9898 108.7898)
 		(end 114.0000 108.0000)
-		(width 0.3)
+		(width 0.5)
 		(layer "F.Cu")
 		(net 1)
 	)
 	(segment
+		(start 105.0000 113.7700)
+		(end 105.4057 114.6000)
+		(width 0.5)
+		(layer "F.Cu")
+		(net 3)
+	)
+	(segment
+		(start 105.4057 114.6000)
+		(end 106.4696 114.2507)
+		(width 0.5)
+		(layer "F.Cu")
+		(net 3)
+	)
+	(segment
+		(start 106.4696 114.2507)
+		(end 109.2850 117.6007)
+		(width 0.5)
+		(layer "F.Cu")
+		(net 3)
+	)
+	(segment
+		(start 109.2850 117.6007)
+		(end 115.3211 118.4500)
+		(width 0.5)
+		(layer "F.Cu")
+		(net 3)
+	)
+	(segment
+		(start 115.3211 118.4500)
+		(end 116.3000 117.6000)
+		(width 0.5)
+		(layer "F.Cu")
+		(net 3)
+	)
+	(segment
+		(start 116.3000 117.6000)
+		(end 116.0000 117.0000)
+		(width 0.5)
+		(layer "F.Cu")
+		(net 3)
+	)
+	(segment
+		(start 116.0000 117.0000)
+		(end 117.8000 115.2000)
+		(width 0.5)
+		(layer "F.Cu")
+		(net 3)
+	)
+	(segment
+		(start 117.8000 115.2000)
+		(end 122.0000 115.2000)
+		(width 0.5)
+		(layer "F.Cu")
+		(net 3)
+	)
+	(segment
+		(start 122.0000 115.2000)
+		(end 123.8527 114.0080)
+		(width 0.5)
+		(layer "B.Cu")
+		(net 3)
+	)
+	(segment
+		(start 123.8527 114.0080)
+		(end 124.5665 114.0012)
+		(width 0.5)
+		(layer "B.Cu")
+		(net 3)
+	)
+	(segment
+		(start 124.5665 114.0012)
+		(end 125.0000 113.7700)
+		(width 0.5)
+		(layer "B.Cu")
+		(net 3)
+	)
+	(via
+		(at 122.0000 115.2000)
+		(size 0.6)
+		(drill 0.3)
+		(layers "F.Cu" "B.Cu")
+		(net 3)
+	)
+	(segment
 		(start 116.0000 108.0000)
-		(end 114.0000 110.0000)
-		(width 0.3)
-		(layer "F.Cu")
-		(net 2)
-	)
-	(segment
-		(start 114.0000 110.0000)
-		(end 114.0000 117.0000)
-		(width 0.3)
-		(layer "F.Cu")
-		(net 2)
-	)
-	(segment
-		(start 116.0000 108.0000)
-		(end 116.5000 108.6000)
-		(width 0.3)
-		(layer "F.Cu")
-		(net 2)
-	)
-	(segment
-		(start 116.5000 108.6000)
-		(end 119.1000 111.2000)
-		(width 0.3)
-		(layer "F.Cu")
-		(net 2)
-	)
-	(segment
-		(start 119.1000 111.2000)
-		(end 124.2000 111.2000)
-		(width 0.3)
-		(layer "F.Cu")
-		(net 2)
-	)
-	(segment
-		(start 124.2000 111.2000)
+		(end 116.9774 107.8774)
+		(width 0.5)
+		(layer "F.Cu")
+		(net 2)
+	)
+	(segment
+		(start 116.9774 107.8774)
+		(end 117.2774 107.5774)
+		(width 0.5)
+		(layer "F.Cu")
+		(net 2)
+	)
+	(segment
+		(start 117.2774 107.5774)
+		(end 120.9000 107.1000)
+		(width 0.5)
+		(layer "F.Cu")
+		(net 2)
+	)
+	(segment
+		(start 120.9000 107.1000)
+		(end 124.2000 110.4000)
+		(width 0.5)
+		(layer "B.Cu")
+		(net 2)
+	)
+	(segment
+		(start 124.2000 110.4000)
 		(end 125.0000 111.2300)
-		(width 0.3)
-		(layer "F.Cu")
-		(net 2)
-	)
+		(width 0.5)
+		(layer "B.Cu")
+		(net 2)
+	)
+	(via
+		(at 120.9000 107.1000)
+		(size 0.6)
+		(drill 0.3)
+		(layers "F.Cu" "B.Cu")
+		(net 2)
+	)
