File: boards/01-voltage-divider/output/voltage_divider.kicad_pcb (KiCad board)
At the start: 2 copper layers, 30 x 25 mm, 4 parts, among them J1 Conn_01x02, J2 Conn_01x02

Commit message: fix(board-01): refresh to current main; eliminate VIN/+5V schematic drift (#3291)
Board 01 (voltage-divider) is the gold-standard fleet board per #2394,
but `kct fleet status` was reporting STALE artifacts and a schematic
drift (`3 nets in schematic, 3 in PCB`):

  schematic nets: {+5V, GND, VOUT}   <- stock KiCad power:+5V symbol
  PCB nets:       {VIN, GND, VOUT}   <- project.kct interface name

The PCB net name (`VIN`) matched project.kct's `interfaces.VIN` while
the schematic emitted KiCad's hard-coded `+5V` from `power:+5V`. Result:
the same physical rail had two names, and the source-drift gate in
`fleet_cmd._detect_source_drift` correctly refused to ship the board.

Fixes
-----

* `boards/01-voltage-divider/generate_design.py`
  - Replace `add_power("power:+5V", ...)` with the synthesized
    `add_pwr_symbol("VIN", ...)` (see `elements_mixin.py:_PWR_SYNTH_LIB_PREFIX`).
    The synthesized library `kicad_tools_pwr:VIN` publishes `VIN` as the
    global net name, eliminating the rail-name drift end-to-end.
  - Plumb a `value` parameter through `generate_connector` so J1/J2 emit
    the schematic-side values `IN`/`OUT` on F.Fab instead of the generic
    `Conn_01x02`. Eliminates a spurious "value mismatch" from
    `kct sync --analyze`.

* `src/kicad_tools/schema/bom.py` (`BOMItem.is_power_symbol`)
  - Recognize `kicad_tools_pwr:` synthesized rails and the legacy `#PWR`
    reference prefix as power symbols, alongside stock `power:`.
    Previously the synthesized VIN symbol leaked into BOM extraction as
    a "real" item.

* `src/kicad_tools/export/bom_formats.py` (`BOMFormatter.filter_items`)
  - Drop virtual items (power symbols, in_bom=False) from the emitted
    CSV. Previously only DNP items were filtered; the synthesized VIN
    rail was reaching `bom_jlcpcb.csv` and triggering a BOM/PCB
    reference-mismatch failure in the export preflight.

Regression tests
----------------

New `tests/test_board_01_ship_ready.py` pins four invariants:

  1. Schematic-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
Parts:
- J1: value Conn_01x02 -> IN
- J2: value Conn_01x02 -> OUT
Changed lines of the file:
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@@
       (effects (font (size 1 1) (thickness 0.15)))
     )
-    (fp_text value "Conn_01x02" (at 0 4) (layer "F.Fab")
+    (fp_text value "IN" (at 0 4) (layer "F.Fab")
       (effects (font (size 1 1) (thickness 0.15)))
     )
@@
       (effects (font (size 1 1) (thickness 0.15)))
     )
-    (fp_text value "Conn_01x02" (at 0 4) (layer "F.Fab")
+    (fp_text value "OUT" (at 0 4) (layer "F.Fab")
       (effects (font (size 1 1) (thickness 0.15)))
     )
