File: boards/05-bldc-motor-controller/output/bldc_controller.kicad_pcb (KiCad board)
At the start: 2 copper layers, 80 x 100 mm, 55 parts, among them J1 Power Input, J2 Motor Output, J3 Hall Sensors, J4 SWD-6, Q1 IRLZ44N, Q2 IRLZ44N, Q3 IRLZ44N, Q4 IRLZ44N, Q5 IRLZ44N, Q6 IRLZ44N, U1 LM2596-5.0, U10 STM32G431K8Tx, U2 AMS1117-3.3, U3 DRV8301, Y1 8MHz

Commit message: fix(boards/05): full U3 DRV8301 schematic symbol swap with layout refactor
Issue #3384 (PR #3388) reconciled the BOM/PCB/schematic-value triangle
around U3 and shipped the project-local board05_custom:DRV8301 symbol
library (57-pin HTSSOP-56), but deferred the schematic-side swap because
naïvely placing the new symbol at the historical X_GATE_DRV=280
silently bridged AGND (pin 28) to +3.3V via a J3 Hall-connector column
wire that ran through the DRV8301 left-edge pin lines at x=265.43.

This PR completes the swap:

* design.py now registers the project-local symbol library via the
  Schematic(local_symbol_libs=[...]) param and places U3 directly via
  add_symbol("board05_custom:DRV8301", ...), bypassing GateDriverBlock
  (which hard-codes Driver_Motor:DRV8308).  U3's bootstrap caps
  (C12-C14) and bypass caps (C15-C16) are now created via the existing
  factory helpers + Device:C symbols rather than as block side-effects.

* U3 is placed at (355, 145) -- well east of J3's column wires at
  x=265.43 (the original AGND-vs-+3.3V short) AND clear of R22's
  output stub at (332.74, 123.19) (the secondary GND-vs-GATE_CH
  short that would have hit if U3 sat at x=350).

* All 57 DRV8301 pins now emit per-pin stub wires + labels via
  _emit_pin_net_stub for pins 1-56 and a manual vertical stub for
  pin 57 (PowerPAD, GND).  Net mapping mirrors DRV8301_PINS in the
  PCB-side block.

* Replaces tests/test_board_05_drv8308_pin_nets.py with
  tests/test_board_05_drv8301_pin_nets.py, holding the
  DRV8301-symbol shape, label-on-wire invariant, and the
  AGND-must-be-GND / PWRGD-must-be-+3.3V anti-regression assertion.

Sync-netlist drift on U3: 41 (DRV8308 schematic) -> 19 (this PR).
The 19 remaining U3 mismatches are pure rail-name normalizations
("+3.3V" -> "+3V3", "VMOTOR" -> "+24V") that affect every component
on those rails (J3.4, J4.1, U10.1, etc.) -- a separate global
schematic vs power-symbol naming concern, NOT a U3 pinout error.

ERC: 17 -> 16 violations (1 new lib_sym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
Routing:
- removed copper zone on F.Cu, net +3.3V
- removed copper zone on F.Cu, net +5V
- removed copper zone on B.Cu, net GND
- removed copper zone on F.Cu, net PWR_LED
- removed copper zone on F.Cu, net VMOTOR

Commit message: fix(boards/05): rail-name normalization (+3.3V/+3V3, VMOTOR/+24V) (#3396)
Closes #3393 and finalizes #3384.

The 19 residual U3 pad changes reported by `kct pcb sync-netlist` (and the
additional rail-rename mismatches on J3.4/J4.1/U10.1/R30-32/C6-9/etc.) were
caused by the schematic publishing `+3V3` (from the `power:+3V3` symbol) and
`+24V` (from `power:+24V`) while the PCB NETS dict used the verbose
`"+3.3V"` and the descriptive `"VMOTOR"`.  Stock-KiCad power symbols
always publish their global net name, so kicad-cli always wrote the
schematic netlist with the +24V/+3V3 names — the PCB-side dict was the
authoritative drift source.

Lock-step rename:
* `boards/05-bldc-motor-controller/design.py`:
  - Rail net_labels updated: `net_label="VMOTOR"` -> `"+24V"`,
    `net_label="+3.3V"` -> `"+3V3"`.
  - `NETS` dict: key `"VMOTOR"` -> `"+24V"`, key `"+3.3V"` -> `"+3V3"`.
  - All component-side net string references updated in lock-step
    (J1/J3/J4 pin headers, U1/U2/U3 regulator pin_nets, U10 deferred
    label list, MOSFET drains, bootstrap caps, decoupling caps).
  - Python identifiers `RAIL_VMOTOR` / `RAIL_3V3` and
    `DRV8301_SCHEMATIC_PIN_NETS` dict name are unchanged (they are
    code-level names, not net strings).
* Routed PCB in-place rename:
  - Net declarations `(net 1 "VMOTOR")` -> `(net 1 "+24V")`,
    `(net 3 "+3.3V")` -> `(net 3 "+3V3")`.
  - Pad-level net references on every footprint.
  - Zone net references.
  - Trace geometry untouched -- this is a pure relabel.  Re-routing
    the board from scratch under the current `--backend python`
    pipeline introduces 10 `clearance_segment_segment` + 8
    `clearance_segment_via` violations that the hot-spot regression
    test (`test_committed_pcb_has_no_segment_segment_or_segment_via`)
    forbids.  Preserving the historical routed geometry keeps the
    hot-spot test green AND delivers the rail-rename fix (the issue's
    primary objective) in a single atomic commit.
* Unrouted PCB and schematic regenera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
Connections:
- net +3.3V renamed +3V3
- net VMOTOR renamed +24V
Routing:
- added copper zone on F.Cu, net +24V
- added copper zone on F.Cu, net +3V3
- added copper zone on F.Cu, net +5V
- added copper zone on B.Cu, net GND
- added copper zone on F.Cu, net PWR_LED
