File: boards/external/softstart/output/softstart.kicad_sch (KiCad schematic)
At the start: 74 parts, among them J1 AC_INPUT, J2 AC_OUTPUT, J3 SCAP_POS, J4 SCAP_NEG, J5 SWD-6, Q1A IRFB4110, Q1B IRFB4110, Q2A IRFB4110, Q2B IRFB4110, Q5 AO3400, Q6 AO3400, Q7 2N7002, Q8 2N7002, SW1 RESET, U1 STM32G031K8T6, U2 H11AA1, U3 INA180A3, U4 XC6206-3.3V, U5 UCC27211, U6 UCC27211, U7 LM393, U8 MCP6001, U9 LM7812

Commit message: fix(softstart): reconcile PCB-schematic sync drift to the routed PCB
Aligns the softstart schematic generator to the routed PCB so the
recipe emits a schematic and PCB whose component sets agree:

- 8 decoupling caps (C1/C2/C3/C8/C30/C31/C33/C34) now use an explicit
  C_0805_2012Metric footprint instead of auto_footprint (which resolved
  100nF parts to 0402), matching the PCB-side generate_cap_0805.
- 4 gate-clamp TVS diodes (D_TVS1-4) switch to Diode_SMD:D_SMA to match
  the routed PCB's generate_sma_tvs (DO-214AC land for the SMBJ clamp).
- 14 value mismatches reconciled to the manufacturable PCB BOM values
  (D1=DB107, D2=LED, J1-J4=TB, J5=SWD, R1=1M, R20/R21="100R 5W",
  R25/R27=270k, R26/R28=9.1k E-series parts).

Mounting holes (MH1-4) legitimately have no schematic symbol, so the
reconciler now filters mechanical mounting holes from the PCB component
set before drift analysis -- they no longer register as benign-but-noisy
PCB-only drift on any board.

kct sync --analyze now reports IN SYNC (0 value, 0 footprint, 0 PCB-only)
for the softstart schematic against both the unrouted and routed PCBs,
and kct check no longer prints the "PCB out of sync" warning.

Closes #3496

Co-Authored-By: Claude Opus 4.7 <noreply@anthropic.com>
Parts:
- C1, C2, C3, C30, C31, C33, C34, C8: footprint Capacitor_SMD:C_0402_1005Metric -> Capacitor_SMD:C_0805_2012Metric
- D1: value RB157 -> DB107
- D2: value STATUS -> LED
- D_TVS1, D_TVS2, D_TVS3, D_TVS4: footprint Diode_SMD:D_SMB -> Diode_SMD:D_SMA
- J1: value AC_INPUT -> TB
- J2: value AC_OUTPUT -> TB
- J3: value SCAP_POS -> TB
- J4: value SCAP_NEG -> TB
- J5: value SWD-6 -> SWD
- R1: value 990.0k -> 1M
- R20, R21: value 100R -> 100R 5W
- R25, R27: value 290.0k -> 270k
- R26, R28: value 10k -> 9.1k
