File: boards/external/softstart/output/softstart.kicad_pcb (KiCad board)
At the start: 2 copper layers, 150 x 100 mm, 78 parts, among them J1 TB, J2 TB, J3 TB, J4 TB, J5 SWD, Q1A IRFB4110, Q1B IRFB4110, Q2A IRFB4110, Q2B IRFB4110, Q5 AO3400, Q6 AO3400, Q7 2N7002, Q8 2N7002, SW1 RESET, U1 STM32G031K8T6, U2 H11AA1, U3 INA180A3, U4 XC6206-3.3V, U5 UCC27211, U6 UCC27211, U7 LM393, U8 MCP6001, U9 LM7812

Commit message: feat(pcb): add page_fit to size sheet to board + center, apply to all boards
Add PCB.page_fit(margin=5.0) which rewrites the (paper ...) node to a tight
(paper "User" W H) sized to the Edge.Cuts bbox plus a uniform margin and
translates every board item (footprints, segments, vias, zones incl.
filled_polygons, gr_* graphics, text) so the board is centered with that
margin. Pure geometric translate — relative geometry, routing and DRC
validity are preserved, no re-route needed.

Expose it as `kct pcb page-fit <pcb> [-o out] [--margin] [--dry-run]` and
wire a PAGE_FIT build step (after stitch, before verify/export) so future
boards are centered too. Apply page_fit to all demo boards (00-07 +
external/softstart), both routed and unrouted PCBs, so the committed
layouts fill + center the KiCanvas viewer instead of sitting tiny in an A4
page. Boards 00/01 stay DRC-clean (0 errors); no board's DRC count changed.

Co-Authored-By: Claude Opus 4.7 <noreply@anthropic.com>
Parts:
- moved C1 134.4 mm to (90.0, 69.0)
- moved C2 134.4 mm to (55.0, 92.0)
- moved C20 134.4 mm to (60.0, 41.0)
- moved C21 134.4 mm to (65.0, 41.0)
- moved C22 134.4 mm to (70.0, 41.0)
- moved C23 134.4 mm to (60.0, 73.0)
- moved C24 134.4 mm to (65.0, 73.0)
- moved C25 134.4 mm to (70.0, 73.0)
- moved C3 134.4 mm to (55.0, 95.0)
- moved C30 134.4 mm to (135.0, 63.0)
- moved C31 134.4 mm to (140.0, 61.0)
- moved C32 134.4 mm to (149.0, 17.0)
- moved C33 134.4 mm to (149.0, 23.0)
- moved C34 134.4 mm to (110.0, 65.0)
- moved C4 134.4 mm to (55.0, 98.0)
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
Commit message: fix(pcb): page-fit routed boards only; revert unrouted sources (refs #3714)
page_fit was applied to and committed for the UNROUTED board sources too.
Because the autorouter is absolute-grid-position-dependent, translating the
unrouted boards changed routing outcomes and turned CI red on three jobs:
- Test: board-02 re-route produced a platform-specific segment count.
- Diff-Pair (06) / Match-Group (07): re-routing the moved unrouted boards
  fractured plane nets under the copper-union pour audit (#3509/#3617).

page_fit is a pure post-route translation, so it must touch the ROUTED
output only:
- Revert every unrouted boards/*/output/<name>.kicad_pcb to origin/main
  (byte-identical); keep the page-fitted *_routed.kicad_pcb (gallery/viewer).
- Revert tests/router/test_board02_manufacturable_baseline.py to main
  (unrouted board-02 unchanged -> reproduces main's result).
- Build hook: _run_step_page_fit now operates on the routed PCB only and
  skips cleanly when no routed output exists, instead of falling back to and
  persisting a page-fit unrouted PCB.

Retains the sound geometry fixes (translation-invariant
point_to_segment_distance, _format_coord_mm, diffpair +1e-6 window tolerance).

Co-Authored-By: Claude Opus 4.7 <noreply@anthropic.com>
Parts:
- moved C1 134.4 mm to (185.0, 164.0)
- moved C2 134.4 mm to (150.0, 187.0)
- moved C20 134.4 mm to (155.0, 136.0)
- moved C21 134.4 mm to (160.0, 136.0)
- moved C22 134.4 mm to (165.0, 136.0)
- moved C23 134.4 mm to (155.0, 168.0)
- moved C24 134.4 mm to (160.0, 168.0)
- moved C25 134.4 mm to (165.0, 168.0)
- moved C3 134.4 mm to (150.0, 190.0)
- moved C30 134.4 mm to (230.0, 158.0)
- moved C31 134.4 mm to (235.0, 156.0)
- moved C32 134.4 mm to (244.0, 112.0)
- moved C33 134.4 mm to (244.0, 118.0)
- moved C34 134.4 mm to (205.0, 160.0)
- moved C4 134.4 mm to (150.0, 193.0)
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