File: boards/06-diffpair-test/output/diffpair_test.kicad_sch (KiCad schematic)
At the start: 7 parts, among them J1 USB-C, J3 MiniPCIe, J4 FFC4, U1 QFN32_USB2, U2 BGA49_USB3, U3 QFP48_PCIe, U4 QFN24_MIPI

Commit message: feat: prepare real demo boards and verified gallery releases
Redesign the controller, LVDS and SDRAM demos around real components and
ship checked assembly packages for boards 00-07, including firmware,
procurement reviews and hash-bound manufacturing evidence.

Add readiness reporting and gallery gates, scoped Cloudflare account
validation, and the routing, geometry, fabrication-rule, cache, LVS and
stripline fixes surfaced during the manufacturing audit.

Scaffold precision acquisition demo 08 and develop the real USB-C PD
power demo 09 with circuit checks, telemetry tests and saved routing
investigations. Keep incomplete examples explicitly blocked.

Preserve exact board bytes in Git and include hash-bound release renders.
Freeze the historical 32-pad joystick router fixture separately from the
real 44-pin design (Refs #5042).

Retire legacy manufacturing error allowances, point release-gate tests at
the real outputs, and run board04's scoped paid-drill validator in CI.
Keep original silkscreen defects as historical detector witnesses.
Parts:
- removed J1: USB-C, Connector_USB:USB_C_Receptacle_USB2.0, symbol diffpair_lvs:USBC_SRC
- removed J3: MiniPCIe, Connector_PCIE:PCIE_Mini_Edge, symbol diffpair_lvs:MINIPCIE_SRC
- removed J4: FFC4, Connector_FFC:FFC_4P_0.5mm, symbol diffpair_lvs:FFC_SRC
- removed U1: QFN32_USB2, Package_DFN_QFN:QFN-32-1EP_5x5mm_P0.5mm, symbol diffpair_lvs:QFN32_USB2
- removed U2: BGA49_USB3, Package_BGA:BGA-49_5.0x5.0mm_Layout7x7_P0.5mm, symbol diffpair_lvs:BGA49_USB3
- removed U3: QFP48_PCIe, Package_QFP:LQFP-48_7x7mm_P0.5mm, symbol diffpair_lvs:QFP48_PCIE
- removed U4: QFN24_MIPI, Package_DFN_QFN:QFN-24-1EP_4x4mm_P0.5mm, symbol diffpair_lvs:QFN24_MIPI
- added C1: 1nF, Capacitor_SMD:C_0603_1608Metric, symbol lvds_demo:C1
- added C10: 100nF, Capacitor_SMD:C_0603_1608Metric, symbol lvds_demo:C10
- added C11: 1nF, Capacitor_SMD:C_0603_1608Metric, symbol lvds_demo:C11
- added C12: 100nF, Capacitor_SMD:C_0603_1608Metric, symbol lvds_demo:C12
- added C13: 1nF, Capacitor_SMD:C_0603_1608Metric, symbol lvds_demo:C13
- added C14: 100nF, Capacitor_SMD:C_0603_1608Metric, symbol lvds_demo:C14
- added C15: 1nF, Capacitor_SMD:C_0603_1608Metric, symbol lvds_demo:C15
- added C16: 100nF, Capacitor_SMD:C_0603_1608Metric, symbol lvds_demo:C16
- added C17: 10uF, Capacitor_SMD:C_0805_2012Metric, symbol lvds_demo:C17
- added C2: 100nF, Capacitor_SMD:C_0603_1608Metric, symbol lvds_demo:C2
- added C3: 1nF, Capacitor_SMD:C_0603_1608Metric, symbol lvds_demo:C3
- added C4: 100nF, Capacitor_SMD:C_0603_1608Metric, symbol lvds_demo:C4
- added C5: 1nF, Capacitor_SMD:C_0603_1608Metric, symbol lvds_demo:C5
- added C6: 100nF, Capacitor_SMD:C_0603_1608Metric, symbol lvds_demo:C6
- added C7: 1nF, Capacitor_SMD:C_0603_1608Metric, symbol lvds_demo:C7
- added C8: 100nF, Capacitor_SMD:C_0603_1608Metric, symbol lvds_demo:C8
- added C9: 1nF, Capacitor_SMD:C_0603_1608Metric, symbol lvds_demo:C9
- added J1: 3.3V regulated input, Connector_PinHeader_2.54mm:PinHeader_1x02_P2.54mm_Vertical, symbol lvds_demo:J1
- added J2: IN1-4 / GND, Connector_PinHeader_2.54mm:PinHeader_1x08_P2.54mm_Vertical, symbol lvds_demo:J2
- added J3: OUT1-4 / GND, Connector_PinHeader_2.54mm:PinHeader_1x08_P2.54mm_Vertical, symbol lvds_demo:J3
- added R1: 100, Resistor_SMD:R_0603_1608Metric, symbol lvds_demo:R1
- added R2: 100, Resistor_SMD:R_0603_1608Metric, symbol lvds_demo:R2
- added R3: 100, Resistor_SMD:R_0603_1608Metric, symbol lvds_demo:R3
- added R4: 100, Resistor_SMD:R_0603_1608Metric, symbol lvds_demo:R4
- added R5: 100k, Resistor_SMD:R_0603_1608Metric, symbol lvds_demo:R5
- added R6: 100k, Resistor_SMD:R_0603_1608Metric, symbol lvds_demo:R6
- added R7: 100k, Resistor_SMD:R_0603_1608Metric, symbol lvds_demo:R7
- added R8: 100k, Resistor_SMD:R_0603_1608Metric, symbol lvds_demo:R8
- added U1: SN65LVDS1DR, Package_SO:SOIC-8_3.9x4.9mm_P1.27mm, symbol lvds_demo:U1
- added U2: SN65LVDS2DR, Package_SO:SOIC-8_3.9x4.9mm_P1.27mm, symbol lvds_demo:U2
- added U3: SN65LVDS1DR, Package_SO:SOIC-8_3.9x4.9mm_P1.27mm, symbol lvds_demo:U3
- added U4: SN65LVDS2DR, Package_SO:SOIC-8_3.9x4.9mm_P1.27mm, symbol lvds_demo:U4
- added U5: SN65LVDS1DR, Package_SO:SOIC-8_3.9x4.9mm_P1.27mm, symbol lvds_demo:U5
- added U6: SN65LVDS2DR, Package_SO:SOIC-8_3.9x4.9mm_P1.27mm, symbol lvds_demo:U6
- added U7: SN65LVDS1DR, Package_SO:SOIC-8_3.9x4.9mm_P1.27mm, symbol lvds_demo:U7
- added U8: SN65LVDS2DR, Package_SO:SOIC-8_3.9x4.9mm_P1.27mm, symbol lvds_demo:U8
Connections:
- net +3V3: now also C1.1, C10.1, C11.1, C12.1, C13.1, C14.1, C15.1, C16.1, C17.1, C2.1, C3.1, C4.1, C5.1, C6.1, C7.1, C8.1, C9.1, J1.1, U1.1 (VCC), U2.8 (VCC), U3.1 (VCC), U4.8 (VCC), U5.1 (VCC), U6.8 (VCC), U7.1 (VCC), U8.8 (VCC)
- net GND: now also C1.2, C10.2, C11.2, C12.2, C13.2, C14.2, C15.2, C16.2, C17.2, C2.2, C3.2, C4.2, C5.2, C6.2, C7.2, C8.2, C9.2, J1.2, J2.2, J2.4, J2.6, J2.8, J3.2, J3.4, J3.6, J3.8, R5.2, R6.2, R7.2, R8.2, U1.4 (GND), U2.5 (GND), U3.4 (GND), U4.5 (GND), U5.4 (GND), U6.5 (GND), U7.4 (GND), U8.5 (GND)
- new net IN1: J2.1, R5.1, U1.2 (D)
- new net IN2: J2.3, R6.1, U3.2 (D)
- new net IN3: J2.5, R7.1, U5.2 (D)
- new net IN4: J2.7, R8.1, U7.2 (D)
- new net LVDS1_N: R1.2, U1.8 (Z), U2.1 (B)
- new net LVDS1_P: R1.1, U1.7 (Y), U2.2 (A)
- new net LVDS2_N: R2.2, U3.8 (Z), U4.1 (B)
- new net LVDS2_P: R2.1, U3.7 (Y), U4.2 (A)
- new net LVDS3_N: R3.2, U5.8 (Z), U6.1 (B)
- new net LVDS3_P: R3.1, U5.7 (Y), U6.2 (A)
- new net LVDS4_N: R4.2, U7.8 (Z), U8.1 (B)
- new net LVDS4_P: R4.1, U7.7 (Y), U8.2 (A)
- new net OUT1: J3.1, U2.7 (R)
- new net OUT2: J3.3, U4.7 (R)
- new net OUT3: J3.5, U6.7 (R)
- new net OUT4: J3.7, U8.7 (R)
- no-connect marks 0 -> 24
Other:
- title: Differential Pair Test Board -> Four-channel LVDS link demonstrator
