File: boards/09-usbc-pd-power/output/usbc_pd_power.kicad_pcb (KiCad board)
At the start: 4 copper layers, 100 x 65 mm, 47 parts, among them J1 USB-C PD INPUT, J2 5V OUTPUT, J3 I2C HOST 3V3, Q1 AO4407A, Q2 AO4407A, U1 STUSB4500QTR, U2 TPS54302DDCR, U3 INA226AIDGSR, U4 TLV76033DBZR

Commit message: feat(boards): connect board09 power stage and guard critical routing
Connect boot, feedback, enable, MOSFET drive and force-current paths. Native checks report zero geometry violations, 68 opens and 16 connected critical nets. Resolve native findings by saved UUID and verify that deleting the BOOT trace trips the gate.

Retain a rejected support-net routing experiment with two native violations as evidence for #4991. Validation: 42 focused tests, one native fault-injection regression, ERC, label LVS, critical connectivity and 16 readiness hashes; gallery build passed.
Parts:
- moved C7 3.16 mm to (159.5, 95.5), turned to 180 degrees
- moved R9 2.52 mm to (160.2, 99.0)
Routing:
- net VIN: track 3.98 -> 90.3 mm, vias 0 -> 8
- net PMOS_GATE: track 0.00 -> 54.8 mm, vias 0 -> 4
- net PMOS_SOURCE: track 0.00 -> 47.1 mm
- net VOUT_PRE: track 0.00 -> 46.7 mm, vias 0 -> 2
- net +5V_OUT: track 0.00 -> 45.6 mm, vias 0 -> 6
- net VBUS_FUSED: track 0.00 -> 18.6 mm
- net FB: track 0.00 -> 16.0 mm
- net BUCK_EN: track 0.00 -> 14.8 mm, vias 0 -> 2
- net SW: track 19.3 -> 28.1 mm, vias 6 -> 7
- net LED_A: track 0.00 -> 4.00 mm
- net BOOT_CAP: track 0.00 -> 3.58 mm
- net BOOT: track 0.00 -> 2.33 mm
