File: boards/03-usb-joystick/output/readiness-verification/fill-saved/usb_joystick_routed.kicad_pcb (KiCad board)
At the start: 4 copper layers, 80 x 60 mm, 38 parts, among them J1 USB4085-GF-A, J2 Joystick 5V X Y SW, J3 AVR ISP, SW1 TL3342F160QG, SW2 TL3342F160QG, SW3 TL3342F160QG, SW4 TL3342F160QG, SW5 TL3342F160QG, U1 ATMEGA32U4-AU, U2 USBLC6-2SC6, Y1 8MHz

Commit message: wip(board03): re-derive plan from fresh lattice route (#6394)
Routing:
- net VBUS: track 88.0 -> 217.9 mm, vias 14 -> 17
- net VCC: track 111.7 -> 39.1 mm, vias 24 -> 19
- net BTN4: track 48.9 -> 119.4 mm
- net GND: track 69.0 -> 2.47 mm, vias 32 -> 5
- net BTN3: track 38.8 -> 93.2 mm, vias 3 -> 4
- net RESET: track 59.7 -> 107.7 mm, vias 7 -> 8
- net BTN2: track 61.3 -> 95.4 mm, vias 10 -> 8
- net BTN1: track 41.6 -> 67.8 mm, vias 8 -> 4
- net JOY_BTN: track 72.1 -> 54.4 mm
- net ISP_MOSI: track 25.4 -> 37.3 mm
- net JOY_Y: track 36.7 -> 47.5 mm, vias 8 -> 4
- net XTAL1: track 11.9 -> 18.1 mm
- net USB_CC1: track 16.8 -> 11.2 mm, vias 2 -> 1
- net USB_CC2: track 19.4 -> 14.6 mm, vias 1 -> 0
- net XTAL2: track 10.6 -> 15.3 mm, vias 2 -> 0
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