File: boards/07-matchgroup-test/regression-fixture/matchgroup_test_routed.kicad_pcb (KiCad board)
At the start: 4 copper layers, 110 x 95 mm, 8 parts, among them J1 FFC6_MIPI, J2 HDMI19, J3 ADDR_HDR, U1 QFN48_DDR_CTRL, U2 QFN48_DRAM, U3 QFN24_MIPI, U4 BGA49_HDMI, U5 QFP48_SRAM

Commit message: fix(boards): retune board 03 USB_D and board 07 ADDR_BUS skew in place
Apply kct retune-lengths to the committed board 07 regression fixture
(ADDR_BUS 1.0998 -> 0.0169 mm) and the board 03 routed PCB (USB_D
1.32 -> 0.45 mm), refill zones, and tighten the relaxed test pins.

Part of #6730

Co-Authored-By: Claude Sonnet 5.5 <noreply@anthropic.com>
Routing:
- net A4: track 43.3 -> 44.4 mm
- net A6: track 43.3 -> 44.3 mm
