File: boards/07-matchgroup-test/regression-fixture/matchgroup_test.kicad_pcb (KiCad board)
At the start: 4 copper layers, 110 x 95 mm, 8 parts, among them J1 FFC6_MIPI, J2 HDMI19, J3 ADDR_HDR, U1 QFN48_DDR_CTRL, U2 QFN48_DRAM, U3 QFN24_MIPI, U4 BGA49_HDMI, U5 QFP48_SRAM

Commit message: fix(board07): move U4 TMDS balls to the J2-facing column so TMDS_D0_N routes
Board 07's synthetic BGA sink U4 carried its six HDMI TMDS legs on row B
(B1..B6), one ring inside the perimeter. On the seed-42 re-route
TMDS_D0_N was sealed in at U4.B2 by the neighbouring balls plus the other
TMDS escapes (30/31). Moving the TMDS balls to U4's outer column 1
(A1..F1, the edge facing J2) routes 31/31 with clean copper-LVS, two
consecutive runs byte-identical, and no new pinned-KiCad native DRC
findings (7 skew_out_of_range before and after; the 1 unconnected item
is gone).

Measured candidates (all seed 42, C++ backend, PYTHONHASHSEED=42):
row-B baseline 30/31, A2-only 30/31 (prior note), row A A1..A6 30/31
(seal-in moves to U4.A2 plus two power opens), column 1 A1..F1 31/31,
column 1 G1..B1 31/31. A1..F1 is committed as a recipe constant in both
generators, and the same pad re-binding goes into the regression
fixture's route-input PCB so the Match-Group Routing Regression gate's
re-route sees it (verified 31/31, 0 unallowed findings).

- REQUIRED_SIGNAL_REACH 30 -> 31; the recipe's lvs_ok leg now gates.
- board-07-end-to-end (ci.yml) and local-gate.sh drop the TMDS_D0_N
  known open: plain check_copper_lvs.py, check_net_status.py and
  check_board_00_e2e.py --lvs-only.
- check_matchgroup_coverage.py lists the newly measurable findings on
  the newly routed pair by identity: TMDS_D0 pair skew (#7619),
  TMDS_D0_P/N impedance (#7349), HDMI_TMDS_LANES group skew (#7550).
  TMDS_D1 pair skew (4.968 -> 1.584 mm, no longer via-imbalanced) is
  re-pointed from #7619 to #7550.

Closes #7557

Co-Authored-By: Claude Opus 5.5 (1M context) <noreply@anthropic.com>
Connections:
- U4 pad A1: GND -> TMDS_D0_P
- U4 pad B1: TMDS_D0_P -> TMDS_D0_N
- U4 pad B2: TMDS_D0_N -> GND
- U4 pad B3: TMDS_D1_P -> GND
- U4 pad B4: TMDS_D1_N -> GND
- U4 pad B5: TMDS_D2_P -> GND
- U4 pad B6: TMDS_D2_N -> GND
- U4 pad C1: GND -> TMDS_D1_P
- U4 pad D1: GND -> TMDS_D1_N
- U4 pad E1: GND -> TMDS_D2_P
- U4 pad F1: GND -> TMDS_D2_N
Changed lines of the file:
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@@
       (effects (font (size 1 1) (thickness 0.15)))
     )
-    (pad "A1" smd rect (at -3.810 -3.810) (size 0.450 0.450) (layers "F.Cu" "F.Paste" "F.Mask") (net 3 "GND"))
+    (pad "A1" smd rect (at -3.810 -3.810) (size 0.450 0.450) (layers "F.Cu" "F.Paste" "F.Mask") (net 21 "TMDS_D0_P"))
     (pad "A2" smd rect (at -2.540 -3.810) (size 0.450 0.450) (layers "F.Cu" "F.Paste" "F.Mask") (net 3 "GND"))
     (pad "A3" smd rect (at -1.270 -3.810) (size 0.450 0.450) (layers "F.Cu" "F.Paste" "F.Mask") (net 3 "GND"))
@@
     (pad "A6" smd rect (at 2.540 -3.810) (size 0.450 0.450) (layers "F.Cu" "F.Paste" "F.Mask") (net 3 "GND"))
     (pad "A7" smd rect (at 3.810 -3.810) (size 0.450 0.450) (layers "F.Cu" "F.Paste" "F.Mask") (net 3 "GND"))
-    (pad "B1" smd rect (at -3.810 -2.540) (size 0.450 0.450) (layers "F.Cu" "F.Paste" "F.Mask") (net 21 "TMDS_D0_P"))
-    (pad "B2" smd rect (at -2.540 -2.540) (size 0.450 0.450) (layers "F.Cu" "F.Paste" "F.Mask") (net 22 "TMDS_D0_N"))
-    (pad "B3" smd rect (at -1.270 -2.540) (size 0.450 0.450) (layers "F.Cu" "F.Paste" "F.Mask") (net 23 "TMDS_D1_P"))
-    (pad "B4" smd rect (at 0.000 -2.540) (size 0.450 0.450) (layers "F.Cu" "F.Paste" "F.Mask") (net 24 "TMDS_D1_N"))
-    (pad "B5" smd rect (at 1.270 -2.540) (size 0.450 0.450) (layers "F.Cu" "F.Paste" "F.Mask") (net 25 "TMDS_D2_P"))
-    (pad "B6" smd rect (at 2.540 -2.540) (size 0.450 0.450) (layers "F.Cu" "F.Paste" "F.Mask") (net 26 "TMDS_D2_N"))
+    (pad "B1" smd rect (at -3.810 -2.540) (size 0.450 0.450) (layers "F.Cu" "F.Paste" "F.Mask") (net 22 "TMDS_D0_N"))
+    (pad "B2" smd rect (at -2.540 -2.540) (size 0.450 0.450) (layers "F.Cu" "F.Paste" "F.Mask") (net 3 "GND"))
+    (pad "B3" smd rect (at -1.270 -2.540) (size 0.450 0.450) (layers "F.Cu" "F.Paste" "F.Mask") (net 3 "GND"))
+    (pad "B4" smd rect (at 0.000 -2.540) (size 0.450 0.450) (layers "F.Cu" "F.Paste" "F.Mask") (net 3 "GND"))
+    (pad "B5" smd rect (at 1.270 -2.540) (size 0.450 0.450) (layers "F.Cu" "F.Paste" "F.Mask") (net 3 "GND"))
+    (pad "B6" smd rect (at 2.540 -2.540) (size 0.450 0.450) (layers "F.Cu" "F.Paste" "F.Mask") (net 3 "GND"))
     (pad "B7" smd rect (at 3.810 -2.540) (size 0.450 0.450) (layers "F.Cu" "F.Paste" "F.Mask") (net 3 "GND"))
-    (pad "C1" smd rect (at -3.810 -1.270) (size 0.450 0.450) (layers "F.Cu" "F.Paste" "F.Mask") (net 3 "GND"))
+    (pad "C1" smd rect (at -3.810 -1.270) (size 0.450 0.450) (layers "F.Cu" "F.Paste" "F.Mask") (net 23 "TMDS_D1_P"))
     (pad "C2" smd rect (at -2.540 -1.270) (size 0.450 0.450) (layers "F.Cu" "F.Paste" "F.Mask") (net 1 "+1V2"))
     (pad "C3" smd rect (at -1.270 -1.270) (size 0.450 0.450) (layers "F.Cu" "F.Paste" "F.Mask") (net 2 "+1V8"))
@@
     (pad "C6" smd rect (at 2.540 -1.270) (size 0.450 0.450) (layers "F.Cu" "F.Paste" "F.Mask") (net 2 "+1V8"))
     (pad "C7" smd rect (at 3.810 -1.270) (size 0.450 0.450) (layers "F.Cu" "F.Paste" "F.Mask") (net 3 "GND"))
-    (pad "D1" smd rect (at -3.810 0.000) (size 0.450 0.450) (layers "F.Cu" "F.Paste" "F.Mask") (net 3 "GND"))
+    (pad "D1" smd rect (at -3.810 0.000) (size 0.450 0.450) (layers "F.Cu" "F.Paste" "F.Mask") (net 24 "TMDS_D1_N"))
     (pad "D2" smd rect (at -2.540 0.000) (size 0.450 0.450) (layers "F.Cu" "F.Paste" "F.Mask") (net 2 "+1V8"))
     (pad "D3" smd rect (at -1.270 0.000) (size 0.450 0.450) (layers "F.Cu" "F.Paste" "F.Mask") (net 2 "+1V8"))
@@
     (pad "D6" smd rect (at 2.540 0.000) (size 0.450 0.450) (layers "F.Cu" "F.Paste" "F.Mask") (net 2 "+1V8"))
     (pad "D7" smd rect (at 3.810 0.000) (size 0.450 0.450) (layers "F.Cu" "F.Paste" "F.Mask") (net 3 "GND"))
-    (pad "E1" smd rect (at -3.810 1.270) (size 0.450 0.450) (layers "F.Cu" "F.Paste" "F.Mask") (net 3 "GND"))
+    (pad "E1" smd rect (at -3.810 1.270) (size 0.450 0.450) (layers "F.Cu" "F.Paste" "F.Mask") (net 25 "TMDS_D2_P"))
     (pad "E2" smd rect (at -2.540 1.270) (size 0.450 0.450) (layers "F.Cu" "F.Paste" "F.Mask") (net 2 "+1V8"))
     (pad "E3" smd rect (at -1.270 1.270) (size 0.450 0.450) (layers "F.Cu" "F.Paste" "F.Mask") (net 2 "+1V8"))
@@
     (pad "E6" smd rect (at 2.540 1.270) (size 0.450 0.450) (layers "F.Cu" "F.Paste" "F.Mask") (net 1 "+1V2"))
     (pad "E7" smd rect (at 3.810 1.270) (size 0.450 0.450) (layers "F.Cu" "F.Paste" "F.Mask") (net 3 "GND"))
-    (pad "F1" smd rect (at -3.810 2.540) (size 0.450 0.450) (layers "F.Cu" "F.Paste" "F.Mask") (net 3 "GND"))
+    (pad "F1" smd rect (at -3.810 2.540) (size 0.450 0.450) (layers "F.Cu" "F.Paste" "F.Mask") (net 26 "TMDS_D2_N"))
     (pad "F2" smd rect (at -2.540 2.540) (size 0.450 0.450) (layers "F.Cu" "F.Paste" "F.Mask") (net 3 "GND"))
     (pad "F3" smd rect (at -1.270 2.540) (size 0.450 0.450) (layers "F.Cu" "F.Paste" "F.Mask") (net 3 "GND"))
