File: boards/07-matchgroup-test/output/matchgroup_test.kicad_sch (KiCad schematic)
At the start: 43 parts, among them J1 5V_INPUT, J2 SWD_3V3, J3 UART_3V3, U1 STM32F429ZIT6, U2 IS42S16400J-6TLI-TR, U3 AP2112K-3.3TRG1

Commit message: fix(boards): drop DRAFT from board 07 titles and re-issue readiness
Remove DRAFT/A-draft from the recipe and the hash-bound reviewed PCB titles,
re-pin the fixture manifests, regenerate the published schematic, renders,
PDFs and report via refresh_bundles_6404.py on the pinned KiCad image, and
re-pin readiness.json and board 07's fleet_routers entry.

Closes #7675

Co-Authored-By: Claude Sonnet 5.5 <noreply@anthropic.com>
Other:
- title: Board 07 real SDRAM memory test — DRAFT -> Board 07 real SDRAM memory test
